Commit message: Lab1, zad do 3

File: urdf/planar2dof.urdf (robot description, URDF)
Before this commit: robot planar2dof, 5 links, 4 joints
Links:
- link planar2dof/link_striker_ee: mass 0.1 -> 5

Commit message: proj1 urdf change

File: urdf/planar2dof.urdf (robot description, URDF)
Before this commit: robot planar2dof, 5 links, 4 joints
Links:
- link planar2dof/base_link: mass 1 -> 3
- link planar2dof/link_striker_ee: mass 5 -> 0.8
